Commit message: Add image from launching Moveit

File: urdf/zed2_holder_panda.xacro (robot description, xacro)
@@ -6,9 +6,9 @@
         <origin xyz="0 0 0" rpy="${pi} 0 0"/>
     </joint>
-    <link name="zed2_holder">
+    <link name="zed2_holder" >
         <inertial>
+        <!-- random values -->
             <mass value="0.05"/>
             <origin xyz="0 0 0"/>
-            <!-- This values for inertia are random just for gazebo to accept -->
             <inertia
                 ixx="0.0003947" ixy="0.0" ixz="3.3365e-8"
@@ -21,4 +21,5 @@
             </geometry>
         </visual>
+        <!-- It was colliding with the robot at the mount point. Since it is not extremely relevant, collision was removed
         <collision>
             <geometry>
@@ -26,4 +27,5 @@
             </geometry>
         </collision>
+        -->
     </link>
 </robot>
