Commit message: Addd no gripper camera

File: urdf/camera_no_gripper.xacro (robot description, xacro)
@@ -4,6 +4,5 @@
         <parent link="panda_hand"/>
         <child link="camera_link"/>
-        <origin xyz="-0.097397 0 0.0274111" rpy="0 -0.824473 0"/>
-        <!-- rotation of =90 degress in pitch and +90 yaw from zed2 left optical frame -->
+        <origin xyz="-0.097397 0 0.0274111" rpy="0 -1.35 0"/>
     </joint>
     <link name="camera_link">
@@ -59,5 +58,5 @@
         <sensor name="zed2_left_raw_camera" type="camera">
             <pose> 0 0 0 0 0 0 </pose>
-            <visualize>false</visualize>
+            <visualize>true</visualize>
             <always_on>true</always_on>
             <update_rate>15</update_rate>

File: urdf/panda_camera.urdf.xacro (robot description, xacro)
@@ -3,9 +3,15 @@
   <xacro:include filename="$(find franka_description)/robots/common/franka_robot.xacro"/>
   <!--
-  Camera with less rotation relvative to the end effector
-  If you want the gripper to appear in the camera view, uncomment the followinf two lines and comment the one above
+  Camera with MORE rotation relative to the end effector
   -->
+  <xacro:include filename="$(find franka_zed_gazebo)/urdf/camera_no_gripper.xacro" />
+  <!--
+  Camera with LESS rotation relative to the end effector
+  If you want the gripper to appear in the camera view, uncomment the following two lines and comment the one above
+  -->
+  <!--
   <xacro:include filename="$(find franka_zed_gazebo)/urdf/camera_gripper.xacro" />
   <xacro:include filename="$(find franka_zed_gazebo)/urdf/zed2_holder_panda_gripper.xacro" />
+  -->
   <xacro:arg name="arm_id" default="panda" />
   <xacro:franka_robot arm_id="$(arg arm_id)"
